Commit message: Updates to get a personal project running.

File: robotiq_2f_140_gripper_visualization/urdf/robotiq_arg2f_140_model_macro.xacro (robot description, xacro)
@@ -139,6 +139,16 @@
            <box size="0.03 0.07 0.0075"/>
         </geometry>
-        <material name="">
-          <color rgba="0.9 0.0 0.0 1" />
+        <!--  Allard adding friction -->
+        <surface>
+        <friction>
+          <ode>
+            <mu>1</mu>
+            <mu2>1</mu2>
+          </ode>
+        </friction>
+      </surface>
+      <!-- END friction-->
+        <material name="">
+          <color rgba="0.9 0.0 0.0 .1" />
         </material>
       </collision>
@@ -159,5 +169,5 @@
       <child link="${prefix}${fingerprefix}_inner_knuckle" />
       <axis xyz="1 0 0" />
-      <limit lower="-0.8757" upper="0.8757" velocity="2.0" effort="1000" />
+      <limit lower="-3.14159" upper="3.14159" velocity="2.0" effort="1000" />
       <mimic joint="${prefix}finger_joint" multiplier="-1" offset="0" />
     </joint>
@@ -169,5 +179,5 @@
       <child link="${prefix}${fingerprefix}_inner_finger" />
       <axis xyz="1 0 0" />
-      <limit lower="-0.8757" upper="0.8757" velocity="2.0" effort="1000" />
+      <limit lower="-3.14159" upper="3.14159" velocity="2.0" effort="1000" />
       <mimic joint="${prefix}finger_joint" multiplier="1" offset="0" />
     </joint>
@@ -188,5 +198,5 @@
       <child link="${prefix}left_outer_knuckle" />
       <axis xyz="-1 0 0" />
-      <limit lower="0" upper="0.7" velocity="2.0" effort="1000" />
+      <limit lower="0" upper="0.775" velocity="2.0" effort="1000" />
     </joint>
     <xacro:finger_joints prefix="${prefix}" fingerprefix="left" reflect="1.0"/>
@@ -198,5 +208,5 @@
       <child link="${prefix}right_outer_knuckle" />
       <axis xyz="1 0 0" />
-      <limit lower="-0.725" upper="0.725" velocity="2.0" effort="1000" />
+      <limit lower="-3.14159" upper="3.14159" velocity="2.0" effort="1000" />
     <mimic joint="${prefix}finger_joint" multiplier="-1" offset="0" />
     </joint>

File: robotiq_2f_140_gripper_visualization/urdf/robotiq_arg2f_transmission.xacro (robot description, xacro)
@@ -5,5 +5,5 @@
       <type>transmission_interface/SimpleTransmission</type>
       <joint name="${prefix}finger_joint">
-        <hardwareInterface>PositionJointInterface</hardwareInterface>
+        <hardwareInterface>hardware_interface/PositionJointInterface</hardwareInterface>
       </joint>
       <actuator name="${prefix}finger_joint_motor">
@@ -11,4 +11,33 @@
       </actuator>
     </transmission>
+          <gazebo>
+              <!-- loading plugin: mimic joints works in gazebo now -->
+              <plugin filename="libroboticsgroup_gazebo_mimic_joint_plugin.so" name="${prefix}mimic_robotiq_140_4">
+                  <joint>${prefix}finger_joint</joint>
+                  <mimicJoint>${prefix}right_outer_knuckle_joint</mimicJoint>
+                  <multiplier>-1.0</multiplier>
+              </plugin>
+              <plugin filename="libroboticsgroup_gazebo_mimic_joint_plugin.so" name="${prefix}mimic_robotiq_140_2">
+                  <joint>${prefix}finger_joint</joint>
+                  <mimicJoint>${prefix}left_inner_finger_joint</mimicJoint>
+                  <multiplier>1.0</multiplier>
+                  <!--<offset>0.0</offset>-->
+              </plugin>
+              <plugin filename="libroboticsgroup_gazebo_mimic_joint_plugin.so" name="${prefix}mimic_robotiq_140_1">
+                  <joint>${prefix}finger_joint</joint>
+                  <mimicJoint>${prefix}right_inner_finger_joint</mimicJoint>
+                  <multiplier>1.0</multiplier>
+              </plugin>
+              <plugin filename="libroboticsgroup_gazebo_mimic_joint_plugin.so" name="${prefix}mimic_robotiq_140_3">
+                  <joint>${prefix}finger_joint</joint>
+                  <mimicJoint>${prefix}left_inner_knuckle_joint</mimicJoint>
+                  <multiplier>-1.0</multiplier>
+              </plugin>
+              <plugin filename="libroboticsgroup_gazebo_mimic_joint_plugin.so" name="${prefix}mimic_robotiq_140_5">
+                  <joint>${prefix}finger_joint</joint>
+                  <mimicJoint>${prefix}right_inner_knuckle_joint</mimicJoint>
+                  <multiplier>-1.0</multiplier>
+              </plugin>
+          </gazebo>
   </xacro:macro>
 </robot>

Commit message: Updates

File: robotiq_2f_140_gripper_visualization/urdf/robotiq_arg2f_140_model_macro.xacro (robot description, xacro)
@@ -143,6 +143,6 @@
         <friction>
           <ode>
-            <mu>1</mu>
-            <mu2>1</mu2>
+            <mu>10000</mu>
+            <mu2>10000</mu2>
           </ode>
         </friction>
@@ -198,5 +198,5 @@
       <child link="${prefix}left_outer_knuckle" />
       <axis xyz="-1 0 0" />
-      <limit lower="0" upper="0.775" velocity="2.0" effort="1000" />
+      <limit lower="0" upper="0.85" velocity="2.0" effort="1000" />
     </joint>
     <xacro:finger_joints prefix="${prefix}" fingerprefix="left" reflect="1.0"/>
